File: PassiveIR.sch (KiCad schematic (older format))
At the start: 26 parts, among them U1 LM358, U2 PassiveIR

Commit message: gg
Parts:
- gave numbers to parts that had none: 3
Changed lines of the file:
@@
 Connection ~ 4650 3750
 $Comp
-L Xenir:ESP32-15-PIN U?
+L Xenir:ESP32-15-PIN U3
 U 1 1 6374DF09
 P 9700 3950
-F 0 "U?" H 9099 4976 50  0000 L BNN
+F 0 "U3" H 9099 4976 50  0000 L BNN
 F 1 "ESP32-15-PIN" H 9099 2849 50  0000 L BNN
 F 2 "" H 9100 5150 50  0001 L BNN
@@
 uC-ADC
 $Comp
-L Diode:DZ2S033X0L D?
+L Diode:DZ2S033X0L D1
 U 1 1 6375235E
 P 8600 3900
-F 0 "D?" H 8600 4000 50  0000 C CNN
+F 0 "D1" H 8600 4000 50  0000 C CNN
 F 1 "DZ2S033X0L" H 8600 3800 50  0000 C CNN
 F 2 "Diode_SMD:D_SOD-523" H 8600 3725 50  0001 C CNN
@@
 $EndComp
 $Comp
-L Xenir:Resistor R?
+L Xenir:Resistor R11
 U 1 1 63753D7E
 P 8350 3750
-F 0 "R?" H 8350 3825 28  0000 C CNN
+F 0 "R11" H 8350 3825 28  0000 C CNN
 F 1 "1k" H 8350 3675 28  0000 C CNN
 F 2 "" H 8350 3650 50  0001 C CNN
@@
 	8150 3750 8100 3750
 $Comp
-L power:GND #PWR?
+L power:GND #PWR014
 U 1 1 63756D35
 P 8600 4050
-F 0 "#PWR?" H 8600 3800 50  0001 C CNN
+F 0 "#PWR014" H 8600 3800 50  0001 C CNN
 F 1 "GND" H 8600 3900 50  0000 C CNN
 F 2 "" H 8600 4050 50  0001 C CNN

Commit message: Update PassiveIR.sch
Parts:
- R8: value 56k -> 27k
Changed lines of the file:
@@
 P 5550 4700
 F 0 "R8" H 5400 4750 28  0000 C CNN
-F 1 "56k" H 5700 4750 28  0000 C CNN
+F 1 "27k" H 5700 4750 28  0000 C CNN
 F 2 "" H 5550 4600 50  0001 C CNN
 F 3 "" H 5550 4600 50  0001 C CNN
